Commit message: fix inertial

File: kuka_kr210_support/urdf/kr210k27002_macro.xacro (robot description, xacro)
@@ -4,7 +4,15 @@
   <xacro:arg name="variant" default="" />
   <xacro:property name="variant" value="$(arg variant)"/>
+  <xacro:macro name="null_inertial">
+    <inertial>
+        <origin xyz="0 0 0" rpy="0 0 0"/>
+        <mass value="1"/>
+        <inertia ixx="1.0" ixy="0.0" ixz="0.0" iyy="1.0" iyz="0.0" izz="1.0"/>
+    </inertial>
+</xacro:macro>
   <xacro:macro name="kuka_kr210k27002" params="prefix">
     <!-- links -->
     <link name="${prefix}base_link">
+      <xacro:null_inertial/>
       <visual>
         <origin xyz="0 0 0" rpy="0 0 0"/>
@@ -22,4 +30,5 @@
     </link>
     <link name="${prefix}link_1">
+      <xacro:null_inertial/>
       <visual>
         <origin xyz="0 0 0" rpy="0 0 0"/>
@@ -37,4 +46,5 @@
     </link>
     <link name="${prefix}link_2">
+      <xacro:null_inertial/>
       <visual>
         <origin xyz="0 0 0" rpy="0 0 0"/>
@@ -52,4 +62,5 @@
     </link>
     <link name="${prefix}link_3">
+      <xacro:null_inertial/>
       <visual>
         <origin xyz="0 0 0" rpy="0 0 0"/>
@@ -67,4 +78,5 @@
     </link>
     <link name="${prefix}link_4">
+      <xacro:null_inertial/>
       <visual>
         <origin xyz="0 0 0" rpy="0 0 0"/>
@@ -82,4 +94,5 @@
     </link>
     <link name="${prefix}link_5">
+      <xacro:null_inertial/>
       <visual>
         <origin xyz="0 0 0" rpy="0 0 0"/>
@@ -97,4 +110,5 @@
     </link>
     <link name="${prefix}link_6">
+      <xacro:null_inertial/>
       <visual>
         <origin xyz="0 0 0" rpy="0 0 0"/>

Commit message: working rsi config

File: kuka_kr210_support/urdf/kr210k27002_macro.xacro (robot description, xacro)
@@ -153,5 +153,5 @@
       <parent link="${prefix}link_3"/>
       <child link="${prefix}link_4"/>
-      <axis xyz="0 0 1"/>
+      <axis xyz="-1 0 0"/>
       <limit lower="${radians(-350)}" upper="${radians(350)}" effort="0" velocity="${radians(179)}"/>
     </joint>
@@ -167,5 +167,5 @@
       <parent link="${prefix}link_5"/>
       <child link="${prefix}link_6"/>
-      <axis xyz="0 0 1"/>
+      <axis xyz="-1 0 0"/>
       <limit lower="${radians(-350)}" upper="${radians(350)}" effort="0" velocity="${radians(220)}"/>
     </joint>
